File: sous-vide.sch (KiCad schematic (older format))
At the start: 25 parts, among them J2 Conn_01x02, J3 Conn_01x02, J4 Conn_01x03, J5 Conn_01x02, Q1 2N3904, SW1 SW_Push_Dual, SW2 SW_Push_Dual, U1 node_mcu1.0, U2 RAC01, U3 G5LE, U4 LCD_Backpack

Commit message: added correct potentiometer footprint
Parts:
- removed J4: Conn_01x03, Pin_Headers:Pin_Header_Straight_1x03_Pitch2.54mm, symbol Conn_01x03
- added U5: P090S-04F20BR10K, P090S-04F20BR10K:TRIM_P090S-04F20BR10K, symbol P090S-04F20BR10K
Connections:
- wire segments 62 -> 60
Other:
- moved on the sheet: D3, D4, J3, R7
Changed lines of the file:
@@
 LIBS:node_mcu1
 LIBS:lcd_backpack
+LIBS:P090S-04F20BR10K
 LIBS:sous-vide-cache
 EELAYER 25 0
@@
 Title "sous-vide"
 Date "2017-12-28"
-Rev "0"
+Rev "0.1"
 Comp "peter mitrano"
 Comment1 ""
@@
 L GND #PWR02
 U 1 1 5A459A02
-P 5600 5050
-F 0 "#PWR02" H 5600 4800 50  0001 C CNN
-F 1 "GND" H 5600 4900 50  0000 C CNN
-F 2 "" H 5600 5050 50  0001 C CNN
-F 3 "" H 5600 5050 50  0001 C CNN
-	1    5600 5050
+P 5400 5200
+F 0 "#PWR02" H 5400 4950 50  0001 C CNN
+F 1 "GND" H 5400 5050 50  0000 C CNN
+F 2 "" H 5400 5200 50  0001 C CNN
+F 3 "" H 5400 5200 50  0001 C CNN
+	1    5400 5200
 	0    1    1    0
 $EndComp
@@
 L GND #PWR04
 U 1 1 5A45BBA5
-P 6150 4950
-F 0 "#PWR04" H 6150 4700 50  0001 C CNN
-F 1 "GND" H 6150 4800 50  0000 C CNN
-F 2 "" H 6150 4950 50  0001 C CNN
-F 3 "" H 6150 4950 50  0001 C CNN
-	1    6150 4950
+P 6450 4950
+F 0 "#PWR04" H 6450 4700 50  0001 C CNN
+F 1 "GND" H 6450 4800 50  0000 C CNN
+F 2 "" H 6450 4950 50  0001 C CNN
+F 3 "" H 6450 4950 50  0001 C CNN
+	1    6450 4950
 	0    1    1    0
 $EndComp
@@
 L RESISTOR0402 R7
 U 1 1 5A45BBE8
-P 6350 4950
-F 0 "R7" H 6300 5000 45  0000 L BNN
-F 1 "11k" H 6300 4850 45  0000 L BNN
-F 2 "Resistors_THT:R_Axial_DIN0204_L3.6mm_D1.6mm_P7.62mm_Horizontal" H 6350 5100 20  0001 C CNN
-F 3 "" H 6350 4950 60  0001 C CNN
-F 4 " " H 6350 5150 60  0000 C CNN "Field4"
-	1    6350 4950
+P 6650 4950
+F 0 "R7" H 6600 5000 45  0000 L BNN
+F 1 "11k" H 6600 4850 45  0000 L BNN
+F 2 "Resistors_THT:R_Axial_DIN0204_L3.6mm_D1.6mm_P7.62mm_Horizontal" H 6650 5100 20  0001 C CNN
+F 3 "" H 6650 4950 60  0001 C CNN
+F 4 " " H 6650 5150 60  0000 C CNN "Field4"
+	1    6650 4950
 	-1   0    0    1
 $EndComp
@@
 $EndComp
 Wire Wire Line
-	6700 4050 4650 4050
+	6950 4050 4650 4050
 Wire Wire Line
 	2950 2800 2950 3250
@@
 	2950 3250 3250 3250
 Wire Wire Line
-	6600 4900 6600 5050
-Wire Wire Line
-	4650 4150 5900 4150
+	6850 4900 6850 5050
+Wire Wire Line
+	4650 4150 6250 4150
 Wire Wire Line
 	4750 5350 4750 3650
@@
 	4850 3750 4650 3750
 Wire Wire Line
-	6550 4950 6600 4950
-Connection ~ 6600 4950
+	6850 4950 6850 4950
+Connection ~ 6850 4950
 Wire Wire Line
 	6850 3850 7100 3850
@@
 	2050 3900 2200 3900
 Wire Wire Line
-	6700 4050 6700 5050
-Wire Wire Line
-	4650 4450 6600 4450
-Wire Wire Line
-	6600 4450 6600 4600
-Wire Wire Line
-	5750 4500 5750 4500
-Wire Wire Line
-	5750 4500 5750 4450
-Connection ~ 5750 4450
+	6950 4050 6950 5050
+Wire Wire Line
+	4650 4450 6850 4450
+Wire Wire Line
+	6850 4450 6850 4600
+Wire Wire Line
+	5850 4500 5850 4450
+Connection ~ 5850 4450
 $Comp
 L D D3
 U 1 1 5A44722D
-P 5750 4650
-F 0 "D3" H 5750 4750 50  0000 C CNN
-F 1 "D" H 5750 4550 50  0000 C CNN
-F 2 "Diodes_THT:D_DO-35_SOD27_P7.62mm_Horizontal" H 5750 4650 50  0001 C CNN
-F 3 "https://www.fairchildsemi.com/datasheets/1N/1N914.pdf" H 5750 4650 50  0001 C CNN
-F 4 "1N4148FS-ND" H 5750 4650 60  0001 C CNN "Part #"
-	1    5750 4650
-	0    1    1    0
-$EndComp
-Wire Wire Line
-	5750 4800 5750 5050
-Wire Wire Line
-	5700 4850 5750 4850
-Connection ~ 5750 4850
+P 5850 4650
+F 0 "D3" H 5850 4750 50  0000 C CNN
+F 1 "D" H 5850 4550 50  0000 C CNN
+F 2 "Diodes_THT:D_DO-35_SOD27_P7.62mm_Horizontal" H 5850 4650 50  0001 C CNN
+F 3 "https://www.fairchildsemi.com/datasheets/1N/1N914.pdf" H 5850 4650 50  0001 C CNN
+F 4 "1N4148FS-ND" H 5850 4650 60  0001 C CNN "Part #"
+	1    5850 4650
+	0    1    1    0
+$EndComp
+Wire Wire Line
+	5850 4800 5850 4900
+Wire Wire Line
+	5700 4850 5850 4850
+Connection ~ 5850 4850
 Wire Wire Line
 	6850 3850 6850 3800
@@
 L D D4
 U 1 1 5A45CBFB
-P 6600 4750
-F 0 "D4" H 6600 4850 50  0000 C CNN
-F 1 "D" H 6600 4650 50  0000 C CNN
-F 2 "Diodes_THT:D_DO-35_SOD27_P7.62mm_Horizontal" H 6600 4750 50  0001 C CNN
-F 3 "https://www.fairchildsemi.com/datasheets/1N/1N914.pdf" H 6600 4750 50  0001 C CNN
-F 4 "1N4148FS-ND" H 6600 4750 60  0001 C CNN "Part #"
-	1    6600 4750
+P 6850 4750
+F 0 "D4" H 6850 4850 50  0000 C CNN
+F 1 "D" H 6850 4650 50  0000 C CNN
+F 2 "Diodes_THT:D_DO-35_SOD27_P7.62mm_Horizontal" H 6850 4750 50  0001 C CNN
+F 3 "https://www.fairchildsemi.com/datasheets/1N/1N914.pdf" H 6850 4750 50  0001 C CNN
+F 4 "1N4148FS-ND" H 6850 4750 60  0001 C CNN "Part #"
+	1    6850 4750
 	0    1    1    0
 $EndComp
@@
 $Comp
 L +3.3V #PWR016
-U 1 1 5A4637BE
-P 3150 3950
-F 0 "#PWR016" H 3150 3800 50  0001 C CNN
-F 1 "+3.3V" H 3150 4090 50  0000 C CNN
-F 2 "" H 3150 3950 50  0001 C CNN
-F 3 "" H 3150 3950 50  0001 C CNN
-	1    3150 3950
-	0    -1   -1   0
-$EndComp
-Wire Wire Line
-	3150 3950 3250 3950
-$Comp
-L +3.3V #PWR017
 U 1 1 5A4638F6
 P 1650 3900
-F 0 "#PWR017" H 1650 3750 50  0001 C CNN
+F 0 "#PWR016" H 1650 3750 50  0001 C CNN
 F 1 "+3.3V" H 1650 4040 50  0000 C CNN
 F 2 "" H 1650 3900 50  0001 C CNN
@@
 $EndComp
 $Comp
-L +3.3V #PWR018
+L +3.3V #PWR017
 U 1 1 5A46393A
 P 1650 4300
-F 0 "#PWR018" H 1650 4150 50  0001 C CNN
+F 0 "#PWR017" H 1650 4150 50  0001 C CNN
 F 1 "+3.3V" H 1650 4440 50  0000 C CNN
 F 2 "" H 1650 4300 50  0001 C CNN
@@
 $EndComp
 $Comp
-L +5V #PWR019
+L +5V #PWR018
 U 1 1 5A46409D
 P 4900 3050
-F 0 "#PWR019" H 4900 2900 50  0001 C CNN
+F 0 "#PWR018" H 4900 2900 50  0001 C CNN
 F 1 "+5V" H 4900 3190 50  0000 C CNN
 F 2 "" H 4900 3050 50  0001 C CNN
@@
 $EndComp
 $Comp
-L +5V #PWR020
+L +5V #PWR019
 U 1 1 5A4640F9
 P 6400 2900
-F 0 "#PWR020" H 6400 2750 50  0001 C CNN
+F 0 "#PWR019" H 6400 2750 50  0001 C CNN
 F 1 "+5V" H 6400 3040 50  0000 C CNN
 F 2 "" H 6400 2900 50  0001 C CNN
@@
 	6400 2900 6500 2900
 $Comp
-L +5V #PWR021
+L +5V #PWR020
 U 1 1 5A4658D3
 P 4950 5350
-F 0 "#PWR021" H 4950 5200 50  0001 C CNN
+F 0 "#PWR020" H 4950 5200 50  0001 C CNN
 F 1 "+5V" H 4950 5490 50  0000 C CNN
 F 2 "" H 4950 5350 50  0001 C CNN
@@
 Connection ~ 5900 2600
 $Comp
-L PWR_FLAG #FLG022
+L PWR_FLAG #FLG021
 U 1 1 5A466CF9
 P 5900 2550
-F 0 "#FLG022" H 5900 2625 50  0001 C CNN
+F 0 "#FLG021" H 5900 2625 50  0001 C CNN
 F 1 "PWR_FLAG" H 5900 2700 50  0000 C CNN
 F 2 "" H 5900 2550 50  0001 C CNN
@@
 	5900 2550 5900 2600
 $Comp
-L PWR_FLAG #FLG023
+L PWR_FLAG #FLG022
 U 1 1 5A466F5E
 P 5900 2750
-F 0 "#FLG023" H 5900 2825 50  0001 C CNN
+F 0 "#FLG022" H 5900 2825 50  0001 C CNN
 F 1 "PWR_FLAG" H 5900 2900 50  0000 C CNN
 F 2 "" H 5900 2750 50  0001 C CNN
@@
 	5900 2750 5900 2700
 Wire Wire Line
-	5600 5050 5650 5050
-Wire Wire Line
-	5900 5050 5850 5050
-Wire Wire Line
-	5900 4150 5900 5050
-$Comp
-L Conn_01x03 J4
-U 1 1 5A46C5AC
-P 5750 5250
-F 0 "J4" H 5750 5450 50  0000 C CNN
-F 1 "Conn_01x03" V 5850 5250 50  0000 C CNN
-F 2 "Pin_Headers:Pin_Header_Straight_1x03_Pitch2.54mm" H 5750 5250 50  0001 C CNN
-F 3 "" H 5750 5250 50  0001 C CNN
-	1    5750 5250
-	0    1    1    0
-$EndComp
+	5400 5200 5450 5200
+Wire Wire Line
+	6250 4150 6250 5200
 $Comp
 L Conn_01x02 J5
@@
 L Conn_01x02 J3
 U 1 1 5A46D37D
-P 6700 5250
-F 0 "J3" H 6700 5350 50  0000 C CNN
-F 1 "Conn_01x02" H 6700 5050 50  0000 C CNN
-F 2 "Pin_Headers:Pin_Header_Straight_1x02_Pitch2.54mm" H 6700 5250 50  0001 C CNN
-F 3 "" H 6700 5250 50  0001 C CNN
-	1    6700 5250
+P 6950 5250
+F 0 "J3" H 6950 5350 50  0000 C CNN
+F 1 "Conn_01x02" H 6950 5050 50  0000 C CNN
+F 2 "Pin_Headers:Pin_Header_Straight_1x02_Pitch2.54mm" H 6950 5250 50  0001 C CNN
+F 3 "" H 6950 5250 50  0001 C CNN
+	1    6950 5250
 	0    1    1    0
 $EndComp
@@
 	1650 4300 1650 4500
 $Comp
-L +3.3V #PWR?
+L +3.3V #PWR023
 U 1 1 5A476C4E
 P 3250 3050
-F 0 "#PWR?" H 3250 2900 50  0001 C CNN
+F 0 "#PWR023" H 3250 2900 50  0001 C CNN
 F 1 "+3.3V" H 3250 3190 50  0000 C CNN
 F 2 "" H 3250 3050 50  0001 C CNN
@@
 	0    -1   -1   0
 $EndComp
+$Comp
+L +3.3V #PWR024
+U 1 1 5A4637BE
+P 3150 3950
+F 0 "#PWR024" H 3150 3800 50  0001 C CNN
+F 1 "+3.3V" H 3150 4090 50  0000 C CNN
+F 2 "" H 3150 3950 50  0001 C CNN
+F 3 "" H 3150 3950 50  0001 C CNN
+	1    3150 3950
+	0    -1   -1   0
+$EndComp
+Wire Wire Line
+	3150 3950 3250 3950
+$Comp
+L P090S-04F20BR10K U5
+U 1 1 5A47477A
+P 5850 5200
+F 0 "U5" H 5449 5701 50  0000 L BNN
+F 1 "P090S-04F20BR10K" H 5450 5050 50  0000 L BNN
+F 2 "P090S-04F20BR10K:TRIM_P090S-04F20BR10K" H 5850 5200 50  0001 L BNN
+F 3 "P090S-04F20BR10K" H 5850 5200 50  0001 L BNN
+F 4 "Good" H 5850 5200 50  0001 L BNN "Field4"
+F 5 "Res Conductive Plastic POT 10K Ohm 20% 0.03W 1(Elec)/1(Mech)Turn 6mm (11.4 X 12.65 X 23mm) Pin Bracket Mount/Through ..." H 5850 5200 50  0001 L BNN "Field5"
+F 6 "0.40 USD" H 5850 5200 50  0001 L BNN "Field6"
+F 7 "None" H 5850 5200 50  0001 L BNN "Field7"
+F 8 "TT Electronics/BI" H 5850 5200 50  0001 L BNN "Field8"
+	1    5850 5200
+	1    0    0    -1
+$EndComp
 $EndSCHEMATC
