File: sous-vide.sch (KiCad schematic (older format))
At the start: 23 parts, among them J1 Conn_01x02, J2 Conn_01x02, J3 Conn_01x02, Q1 2N3904, SW1 SW_Push_Dual, SW2 SW_Push_Dual, U1 G5LE, U2 RAC01, U3 node_mcu1.0, U4 P090S, U5 LCD_Backpack

Commit message: add filter capacitor to thermistor
Parts:
- added C1: C, Capacitors_THT:C_Disc_D4.3mm_W1.9mm_P5.00mm, symbol C
Connections:
- net THERMISTOR: now also C1.1
- net at D4.2 (A), J3.2 (Pin_2), R6.2: now also C1.2
Other:
- moved on the sheet: J3
Changed lines of the file:
@@
 L Conn_01x02 J3
 U 1 1 5A46D37D
-P 7500 5350
-F 0 "J3" H 7500 5450 50  0000 C CNN
-F 1 "Conn_01x02" H 7500 5150 50  0000 C CNN
-F 2 "Pin_Headers:Pin_Header_Straight_1x02_Pitch2.54mm" H 7500 5350 50  0001 C CNN
-F 3 "" H 7500 5350 50  0001 C CNN
-	1    7500 5350
+P 8050 5350
+F 0 "J3" H 8050 5450 50  0000 C CNN
+F 1 "Conn_01x02" H 8050 5150 50  0000 C CNN
+F 2 "Pin_Headers:Pin_Header_Straight_1x02_Pitch2.54mm" H 8050 5350 50  0001 C CNN
+F 3 "" H 8050 5350 50  0001 C CNN
+	1    8050 5350
 	1    0    0    -1
 $EndComp
@@
 SW2
 Wire Wire Line
-	6950 5450 7300 5450
+	6950 5450 7450 5450
 Connection ~ 7200 5450
 Wire Wire Line
@@
 Wire Wire Line
 	6650 4300 6650 5350
-Wire Wire Line
-	6650 5350 7300 5350
 Connection ~ 6150 5900
 Wire Wire Line
@@
 NoConn ~ 5550 3300
 NoConn ~ 5650 3300
+$Comp
+L C C1
+U 1 1 5A494F7C
+P 7600 5400
+F 0 "C1" H 7625 5500 50  0000 L CNN
+F 1 "C" H 7625 5300 50  0000 L CNN
+F 2 "Capacitors_THT:C_Disc_D4.3mm_W1.9mm_P5.00mm" H 7638 5250 50  0001 C CNN
+F 3 "" H 7600 5400 50  0001 C CNN
+	1    7600 5400
+	1    0    0    -1
+$EndComp
+Wire Wire Line
+	7450 5250 7850 5250
+Wire Wire Line
+	7850 5250 7850 5350
+Wire Wire Line
+	7450 5550 7850 5550
+Wire Wire Line
+	7850 5550 7850 5450
+Wire Wire Line
+	7450 5450 7450 5550
+Connection ~ 7600 5550
+Wire Wire Line
+	6650 5350 7450 5350
+Wire Wire Line
+	7450 5350 7450 5250
+Connection ~ 7600 5250
 $EndSCHEMATC

Commit message: thermistor test "works"
 - if I understand correctly, R_Ref is calculated to be 1.1k
 - works for the one sample (Temp, ADC) I have
 - removed the 1k resistor on the relay circuit
Parts:
- removed R3: 1.1k, Resistors_THT:R_Axial_DIN0207_L6.3mm_D2.5mm_P10.16mm_Horizontal, symbol RESISTOR0402
- added R7: 1.1k, Resistors_THT:R_Axial_DIN0207_L6.3mm_D2.5mm_P10.16mm_Horizontal, symbol RESISTOR0402
- C1: value C -> 200nF
Connections:
- net THERMISTOR: now also R7.1; no longer J3.1 (Pin_1)
- net at Q1.2 (B): now also U3.26 (D8/GPIO15)
- new net: J3.1 (Pin_1), R7.2
Other:
- moved on the sheet: J3
Changed lines of the file:
@@
-$EndComp
-$Comp
-L RESISTOR0402 R3
-U 1 1 5A45D230
-P 6450 2350
-F 0 "R3" H 6400 2400 45  0000 L BNN
-F 1 "1.1k" H 6400 2250 45  0000 L BNN
-F 2 "Resistors_THT:R_Axial_DIN0207_L6.3mm_D2.5mm_P10.16mm_Horizontal" H 6450 2500 20  0001 C CNN
-F 3 "" H 6450 2350 60  0001 C CNN
-F 4 " " H 6450 2550 60  0000 C CNN "Field4"
-	1    6450 2350
-	0    1    1    0
 $EndComp
 $Comp
@@
 L Conn_01x02 J3
 U 1 1 5A46D37D
-P 8050 5350
-F 0 "J3" H 8050 5450 50  0000 C CNN
-F 1 "Conn_01x02" H 8050 5150 50  0000 C CNN
-F 2 "Pin_Headers:Pin_Header_Straight_1x02_Pitch2.54mm" H 8050 5350 50  0001 C CNN
-F 3 "" H 8050 5350 50  0001 C CNN
-	1    8050 5350
+P 8850 5350
+F 0 "J3" H 8850 5450 50  0000 C CNN
+F 1 "Conn_01x02" H 8850 5150 50  0000 C CNN
+F 2 "Pin_Headers:Pin_Header_Straight_1x02_Pitch2.54mm" H 8850 5350 50  0001 C CNN
+F 3 "" H 8850 5350 50  0001 C CNN
+	1    8850 5350
 	1    0    0    -1
 $EndComp
@@
 	6350 4100 8000 4100
 Wire Wire Line
-	6450 2550 6450 4000
+	6450 2150 6450 4000
 Wire Wire Line
 	6450 4000 6350 4000
@@
 P 7600 5400
 F 0 "C1" H 7625 5500 50  0000 L CNN
-F 1 "C" H 7625 5300 50  0000 L CNN
+F 1 "200nF" H 7625 5300 50  0000 L CNN
 F 2 "Capacitors_THT:C_Disc_D4.3mm_W1.9mm_P5.00mm" H 7638 5250 50  0001 C CNN
 F 3 "" H 7600 5400 50  0001 C CNN
@@
 $EndComp
 Wire Wire Line
-	7450 5250 7850 5250
-Wire Wire Line
-	7850 5250 7850 5350
-Wire Wire Line
-	7450 5550 7850 5550
-Wire Wire Line
-	7850 5550 7850 5450
+	7450 5250 7900 5250
+Wire Wire Line
+	7900 5250 7900 5350
+Wire Wire Line
+	7450 5550 7900 5550
+Wire Wire Line
+	7900 5550 7900 5450
 Wire Wire Line
 	7450 5450 7450 5550
@@
 	7450 5350 7450 5250
 Connection ~ 7600 5250
+$Comp
+L RESISTOR0402 R7
+U 1 1 5A496D58
+P 8100 5350
+F 0 "R7" H 8050 5400 45  0000 L BNN
+F 1 "1.1k" H 8050 5250 45  0000 L BNN
+F 2 "Resistors_THT:R_Axial_DIN0207_L6.3mm_D2.5mm_P10.16mm_Horizontal" H 8100 5500 20  0001 C CNN
+F 3 "" H 8100 5350 60  0001 C CNN
+F 4 " " H 8100 5550 60  0000 C CNN "Field4"
+	1    8100 5350
+	1    0    0    1
+$EndComp
+Wire Wire Line
+	7900 5450 8650 5450
+Wire Wire Line
+	8300 5350 8650 5350
 $EndSCHEMATC

Commit message: ready for Fab!
Parts:
- added J4, J5: Jumper, Pin_Headers:Pin_Header_Straight_1x02_Pitch2.54mm, symbol Conn_01x02
Connections:
- net +5V: now also J4.2 (Pin_2); no longer D2.1 (K), U1.2 (+Coil)
- net at Q1.2 (B), U3.26 (D8/GPIO15): now also J5.2 (Pin_2)
- new net: D2.1 (K), J4.1 (Pin_1), J5.1 (Pin_1), U1.2 (+Coil)
Changed lines of the file:
@@
 L +5V #PWR017
 U 1 1 5A491092
-P 6050 1300
-F 0 "#PWR017" H 6050 1150 50  0001 C CNN
-F 1 "+5V" H 6050 1440 50  0000 C CNN
-F 2 "" H 6050 1300 50  0001 C CNN
-F 3 "" H 6050 1300 50  0001 C CNN
-	1    6050 1300
+P 6050 900
+F 0 "#PWR017" H 6050 750 50  0001 C CNN
+F 1 "+5V" H 6050 1040 50  0000 C CNN
+F 2 "" H 6050 900 50  0001 C CNN
+F 3 "" H 6050 900 50  0001 C CNN
+	1    6050 900
 	1    0    0    -1
 $EndComp
@@
 Text Label 4250 3950 3    60   ~ 0
 SW2
-Wire Wire Line
-	6950 5450 7450 5450
-Connection ~ 7200 5450
-Wire Wire Line
-	5600 1400 6050 1400
-Wire Wire Line
-	6050 1300 6050 1450
-Wire Wire Line
-	5650 1850 6250 1850
-Wire Wire Line
-	6050 1750 6050 1900
-Connection ~ 6050 1400
-Wire Wire Line
-	5600 1600 5650 1600
-Wire Wire Line
-	5650 1600 5650 1850
-Connection ~ 6050 1850
-Connection ~ 3650 2300
-Wire Wire Line
-	3650 2350 3650 2300
-Connection ~ 3650 2200
-Wire Wire Line
-	3650 2150 3650 2200
-Wire Wire Line
-	6100 5900 6200 5900
-Wire Wire Line
-	3550 3550 3700 3550
-Wire Wire Line
-	3550 4150 3700 4150
-Wire Wire Line
-	4100 3550 4450 3550
-Wire Wire Line
-	6350 3550 6350 3800
-Wire Wire Line
-	7800 4300 8000 4300
-Wire Wire Line
-	8000 4400 7550 4400
-Wire Wire Line
-	6350 3550 6850 3550
-Wire Wire Line
-	6900 3900 6350 3900
-Wire Wire Line
-	6500 4400 6500 5500
-Wire Wire Line
-	7800 3800 7800 4300
-Wire Wire Line
-	5200 3300 5350 3300
-Wire Wire Line
-	6650 4300 6650 5350
-Connection ~ 6150 5900
-Wire Wire Line
-	4450 5450 6650 5450
-Wire Wire Line
-	4450 5450 4450 4850
-Wire Wire Line
-	5800 5900 5800 5450
-Connection ~ 5800 5450
-Wire Notes Line
-	2950 2850 2950 750
-Wire Notes Line
-	2950 750  5000 750
-Wire Notes Line
-	5000 750  5000 2850
-Wire Notes Line
-	5000 2850 2950 2850
-Wire Wire Line
-	6500 4400 6350 4400
-Wire Wire Line
-	6650 4300 6350 4300
-Wire Wire Line
-	6350 4200 8000 4200
-Wire Wire Line
-	6350 4100 8000 4100
-Wire Wire Line
-	6450 2150 6450 4000
-Wire Wire Line
-	6450 4000 6350 4000
-Wire Wire Line
-	3500 2200 4350 2200
-Wire Wire Line
-	4000 2200 4000 1500
-Wire Wire Line
-	4200 1600 4200 2550
-Wire Wire Line
-	4200 1600 4350 1600
-Wire Wire Line
-	3500 2300 4200 2300
-Wire Wire Line
-	3500 1400 4350 1400
-Wire Wire Line
-	4000 1500 3500 1500
 $Comp
 L G5LE U1
@@
 	-1   0    0    -1
 $EndComp
-Connection ~ 4000 2200
-Wire Wire Line
-	4200 2550 4350 2550
-Connection ~ 4200 2300
 Text Label 6550 3550 0    60   ~ 0
 RED_LED
@@
 Text Label 6500 5300 1    60   ~ 0
 UESR_POT
-Wire Wire Line
-	5250 5100 5550 5100
-Connection ~ 5350 5100
-Connection ~ 5400 5100
-Connection ~ 5450 5100
-Wire Wire Line
-	4100 4150 4250 4150
-Wire Wire Line
-	4250 4150 4250 3650
-Wire Wire Line
-	4250 3650 4450 3650
 $Comp
 L node_mcu1.0 U3
@@
 	1    0    0    -1
 $EndComp
-Wire Wire Line
-	7450 5250 7900 5250
-Wire Wire Line
-	7900 5250 7900 5350
-Wire Wire Line
-	7450 5550 7900 5550
-Wire Wire Line
-	7900 5550 7900 5450
-Wire Wire Line
-	7450 5450 7450 5550
-Connection ~ 7600 5550
-Wire Wire Line
-	6650 5350 7450 5350
-Wire Wire Line
-	7450 5350 7450 5250
-Connection ~ 7600 5250
 $Comp
 L RESISTOR0402 R7
@@
 	1    0    0    1
 $EndComp
+$Comp
+L Conn_01x02 J5
+U 1 1 5A4AC97D
+P 6600 1200
+F 0 "J5" H 6600 1300 50  0000 C CNN
+F 1 "Jumper" V 6700 1150 50  0000 C CNN
+F 2 "Pin_Headers:Pin_Header_Straight_1x02_Pitch2.54mm" H 6600 1200 50  0001 C CNN
+F 3 "" H 6600 1200 50  0001 C CNN
+	1    6600 1200
+	0    -1   -1   0
+$EndComp
+$Comp
+L Conn_01x02 J4
+U 1 1 5A4ACB3D
+P 5850 1200
+F 0 "J4" H 5850 1300 50  0000 C CNN
+F 1 "Jumper" H 6050 1150 50  0000 C CNN
+F 2 "Pin_Headers:Pin_Header_Straight_1x02_Pitch2.54mm" H 5850 1200 50  0001 C CNN
+F 3 "" H 5850 1200 50  0001 C CNN
+	1    5850 1200
+	-1   0    0    1
+$EndComp
+Wire Wire Line
+	6950 5450 7450 5450
+Connection ~ 7200 5450
+Wire Wire Line
+	5600 1400 6600 1400
+Wire Wire Line
+	6050 1200 6050 1450
+Wire Wire Line
+	5650 1850 6250 1850
+Wire Wire Line
+	6050 1750 6050 1900
+Connection ~ 6050 1400
+Wire Wire Line
+	5600 1600 5650 1600
+Wire Wire Line
+	5650 1600 5650 1850
+Connection ~ 6050 1850
+Connection ~ 3650 2300
+Wire Wire Line
+	3650 2350 3650 2300
+Connection ~ 3650 2200
+Wire Wire Line
+	3650 2150 3650 2200
+Wire Wire Line
+	6100 5900 6200 5900
+Wire Wire Line
+	3550 3550 3700 3550
+Wire Wire Line
+	3550 4150 3700 4150
+Wire Wire Line
+	4100 3550 4450 3550
+Wire Wire Line
+	6350 3550 6350 3800
+Wire Wire Line
+	7800 4300 8000 4300
+Wire Wire Line
+	8000 4400 7550 4400
+Wire Wire Line
+	6350 3550 6850 3550
+Wire Wire Line
+	6900 3900 6350 3900
+Wire Wire Line
+	6500 4400 6500 5500
+Wire Wire Line
+	7800 3800 7800 4300
+Wire Wire Line
+	5200 3300 5350 3300
+Wire Wire Line
+	6650 4300 6650 5350
+Connection ~ 6150 5900
+Wire Wire Line
+	4450 5450 6650 5450
+Wire Wire Line
+	4450 5450 4450 4850
+Wire Wire Line
+	5800 5900 5800 5450
+Connection ~ 5800 5450
+Wire Notes Line
+	2950 2850 2950 750
+Wire Notes Line
+	2950 750  5000 750
+Wire Notes Line
+	5000 750  5000 2850
+Wire Notes Line
+	5000 2850 2950 2850
+Wire Wire Line
+	6500 4400 6350 4400
+Wire Wire Line
+	6650 4300 6350 4300
+Wire Wire Line
+	6350 4200 8000 4200
+Wire Wire Line
+	6350 4100 8000 4100
+Wire Wire Line
+	6450 2150 6450 4000
+Wire Wire Line
+	6450 4000 6350 4000
+Wire Wire Line
+	3500 2200 4350 2200
+Wire Wire Line
+	4000 2200 4000 1500
+Wire Wire Line
+	4200 1600 4200 2550
+Wire Wire Line
+	4200 1600 4350 1600
+Wire Wire Line
+	3500 2300 4200 2300
+Wire Wire Line
+	3500 1400 4350 1400
+Wire Wire Line
+	4000 1500 3500 1500
+Connection ~ 4000 2200
+Wire Wire Line
+	4200 2550 4350 2550
+Connection ~ 4200 2300
+Wire Wire Line
+	5250 5100 5550 5100
+Connection ~ 5350 5100
+Connection ~ 5400 5100
+Connection ~ 5450 5100
+Wire Wire Line
+	4100 4150 4250 4150
+Wire Wire Line
+	4250 4150 4250 3650
+Wire Wire Line
+	4250 3650 4450 3650
+Wire Wire Line
+	7450 5250 7900 5250
+Wire Wire Line
+	7900 5250 7900 5350
+Wire Wire Line
+	7450 5550 7900 5550
+Wire Wire Line
+	7900 5550 7900 5450
+Wire Wire Line
+	7450 5450 7450 5550
+Connection ~ 7600 5550
+Wire Wire Line
+	6650 5350 7450 5350
+Wire Wire Line
+	7450 5350 7450 5250
+Connection ~ 7600 5250
 Wire Wire Line
 	7900 5450 8650 5450
 Wire Wire Line
 	8300 5350 8650 5350
+Wire Wire Line
+	6700 1400 7200 1400
+Wire Wire Line
+	7200 1400 7200 2200
+Wire Wire Line
+	7200 2200 6450 2200
+Connection ~ 6450 2200
+Wire Wire Line
+	6050 900  6050 1100
 $EndSCHEMATC
